Commit message: stereo_vision version 1

File: bumperbot_description/urdf/bumperbot.urdf.xacro (robot description, xacro)
@@ -205,40 +205,45 @@
   </link>
   <joint name="laser_joint" type="fixed">
-    <origin xyz="-0.0050526 -0.0023221 0.1208" rpy="0 0 3.14" />
+    <origin xyz="-0.0050526 -0.0023221 0.1208" rpy="0 0 0" />
     <parent link="base_link" />
     <child link="laser_link" />
     <axis xyz="0 0 0" />
   </joint>
-  <xacro:if value="${camera_model == 'pi_camera'}">
-    <link name="rgb_camera">
-      <mass value="0.0001" />
-      <inertia ixx="0.001" ixy="0.001" ixz="0.001"
-              iyy="0.001" iyz="0.001"
-              izz="0.001" />
-      <visual>
-        <origin rpy="0.0 0.0 0.0" xyz="0.0 0.0 0.0"/>
-        <geometry>
-          <mesh filename="package://bumperbot_description/meshes/pi_camera.STL"/>
-        </geometry>
-        <material name="green"/>
-      </visual>
-      <collision>
-        <origin rpy="0.0 0.0 0.0" xyz="0.0 0.0 0.0"/>
-        <geometry>
-          <mesh filename="package://bumperbot_description/meshes/pi_camera.STL"/>
-        </geometry>
-      </collision>
-    </link>
-    <joint name ="camera_joint" type="fixed">
-      <parent link="base_link"/>
-      <child link = "rgb_camera"/>
-      <origin xyz="0.078 0.0 0.07" rpy="0.0 -0.35 0.0"/>
-    </joint>
-  </xacro:if>
-  <xacro:if value="${camera_model == 'realsense_d435'}">
-    <xacro:sensor_d435 name="rgbd_camera" parent="base_link" use_nominal_extrinsics="$(arg is_sim)">
-      <origin xyz="0.07 0.0 0.08" rpy="0.0 0.0 0.0"/>
-    </xacro:sensor_d435>
-  </xacro:if>
+  <link name="camera_link">
+    <mass value="0.0001" />
+    <inertia ixx="0.001" ixy="0.001" ixz="0.001"
+            iyy="0.001" iyz="0.001"
+            izz="0.001" />
+    <visual>
+      <origin rpy="0.0 0.0 0.0" xyz="0.0 0.0 0.0"/>
+      <geometry>
+        <mesh filename="package://bumperbot_description/meshes/stereo_camera.STL"/>
+      </geometry>
+      <material name="dark_grey"/>
+    </visual>
+    <collision>
+      <origin rpy="0.0 0.0 0.0" xyz="0.0 0.0 0.0"/>
+      <geometry>
+        <mesh filename="package://bumperbot_description/meshes/stereo_camera.STL"/>
+      </geometry>
+    </collision>
+  </link>
+  <joint name ="camera_joint" type="fixed">
+    <parent link="base_link"/>
+    <child link = "camera_link"/>
+    <origin xyz="0.05 0.03 0.095" rpy="0.0 -0.35 0.0"/>
+  </joint>
+  <link name="right_camera_link"/>
+  <joint name ="right_camera_joint" type="fixed">
+    <parent link="camera_link"/>
+    <child link = "right_camera_link"/>
+    <origin xyz="0.0 -0.06 0.0" rpy="0.0 0.0 0.0"/>
+  </joint>
+  <link name="left_camera_link"/>
+  <joint name ="left_camera_joint" type="fixed">
+    <parent link="camera_link"/>
+    <child link = "left_camera_link"/>
+    <origin xyz="0.0 0.0 0.0" rpy="0.0 0.0 0.0"/>
+  </joint>
   <material name="blue">
     <color rgba="0 0 1 1"/>

File: bumperbot_description/urdf/bumperbot_gazebo.xacro (robot description, xacro)
@@ -144,84 +144,55 @@
   </gazebo>
   <!-- RGB Camera -->
-  <xacro:if value="${camera_model == 'pi_camera'}">
-    <gazebo reference="rgb_camera">
-      <sensor name="camera" type="camera">
-        <always_on>true</always_on>
-        <update_rate>30.0</update_rate>
-        <visualize>true</visualize>
-        <topic>/image_raw</topic>
-        <gz_frame_id>/rgb_camera</gz_frame_id>
-        <camera name="camera">
-          <horizontal_fov>1.21126</horizontal_fov>
-          <image>
-            <width>2304</width>
-            <height>1296</height>
-            <format>R8G8B8</format>
-          </image>
-          <distortion>
-            <k1>0.0</k1>
-            <k2>0.0</k2>
-            <k3>0.0</k3>
-            <p1>0.0</p1>
-            <p2>0.0</p2>
-            <center>0.5 0.5</center>
-          </distortion>
-        </camera>
-      </sensor>
-    </gazebo>
-  </xacro:if>
-  <!-- RGBD Camera -->
-  <xacro:if value="${camera_model == 'realsense_d435'}">
-    <gazebo reference="rgbd_camera_link">
-      <sensor name="d435_color" type="camera">
-				<always_on>1</always_on>
-				<update_rate>10</update_rate>
-				<visualize>1</visualize>
-				<topic>/rgbd_camera/image_raw</topic>
-        <gz_frame_id>rgbd_camera_color_optical_frame</gz_frame_id>
-				<camera name="d435">
-					<vertical_fov>1.518</vertical_fov>
-          <horizontal_fov>1.012</horizontal_fov>
-					<image>
-						<width>640</width>
-						<height>480</height>
-						<format>RGB_INT8</format>
-					</image>
-					<clip>
-						<near>0.1</near>
-						<far>100</far>
-					</clip>
-					<noise>
-						<type>gaussian</type>
-						<mean>0</mean>
-						<stddev>0.007</stddev>
-					</noise>
-				</camera>
-			</sensor>
-      <sensor name="d435_depth" type="depth_camera">
-				<always_on>1</always_on>
-				<update_rate>10</update_rate>
-				<visualize>0</visualize>
-				<topic>/rgbd_camera/depth</topic>
-        <gz_frame_id>rgbd_camera_depth_optical_frame</gz_frame_id>
-				<camera name="d435">
-					<vertical_fov>1.518</vertical_fov>
-          <horizontal_fov>1.012</horizontal_fov>
-					<image>
-						<width>640</width>
-						<height>480</height>
-					</image>
-					<clip>
-						<near>0.1</near>
-						<far>100</far>
-					</clip>
-					<noise>
-						<type>gaussian</type>
-						<mean>0</mean>
-						<stddev>0.001</stddev>
-					</noise>
-				</camera>
-			</sensor>
-    </gazebo>
-  </xacro:if>
+  <gazebo reference="left_camera_link">
+    <sensor name="left_camera" type="camera">
+      <always_on>true</always_on>
+      <update_rate>15.0</update_rate>
+      <visualize>true</visualize>
+      <topic>/left_camera/image_raw</topic>
+      <gz_frame_id>/left_camera_link</gz_frame_id>
+      <camera name="left_camera">
+        <horizontal_fov>1.27409</horizontal_fov>
+        <vertical_fov>0.872665</vertical_fov>
+        <image>
+          <width>1280</width>
+          <height>720</height>
+          <format>R8G8B8</format>
+        </image>
+        <distortion>
+          <k1>0.0</k1>
+          <k2>0.0</k2>
+          <k3>0.0</k3>
+          <p1>0.0</p1>
+          <p2>0.0</p2>
+          <center>0.5 0.5</center>
+        </distortion>
+      </camera>
+    </sensor>
+  </gazebo>
+  <gazebo reference="right_camera_link">
+    <sensor name="right_camera" type="camera">
+      <always_on>true</always_on>
+      <update_rate>15.0</update_rate>
+      <visualize>true</visualize>
+      <topic>/right_camera/image_raw</topic>
+      <gz_frame_id>/right_camera_link</gz_frame_id>
+      <camera name="right_camera">
+        <horizontal_fov>1.27409</horizontal_fov>
+        <vertical_fov>0.872665</vertical_fov>
+        <image>
+          <width>1280</width>
+          <height>720</height>
+          <format>R8G8B8</format>
+        </image>
+        <distortion>
+          <k1>0.0</k1>
+          <k2>0.0</k2>
+          <k3>0.0</k3>
+          <p1>0.0</p1>
+          <p2>0.0</p2>
+          <center>0.5 0.5</center>
+        </distortion>
+      </camera>
+    </sensor>
+  </gazebo>
 </robot>
